File: well-siting-meter.sch (EAGLE design)
At the start: 47 parts, among them J2 7805, T1 MOSFET-NCHANNELFQP30N06L, U1 LCD-16X2NOHOLES, U2 ARDUINO_PRO_MINI, U3 EC2, U4 EC2, U5 AD623, U6 AD623, U7 MAX1771

Commit message: rev - mfg files
Parts:
- TM1: PN (none) -> 1528-1997-ND
Changed lines of the file:
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@@
 <part name="GND14" library="SparkFun-Aesthetics" deviceset="GND" device=""/>
 <part name="GND15" library="SparkFun-Aesthetics" deviceset="GND" device=""/>
-<part name="TM1" library="adafruit" deviceset="TRIM" device="3386"/>
+<part name="TM1" library="adafruit" deviceset="TRIM" device="3386">
+<attribute name="PN" value="1528-1997-ND "/>
+</part>
 <part name="L1" library="misc" deviceset="WE-FAMI" device="" value="22uH">
 <attribute name="PN" value="732-7163-ND"/>
@@
 <attribute name="NAME" x="104.14" y="60.96" size="1.778" layer="95" rot="R270"/>
 <attribute name="VALUE" x="104.14" y="60.96" size="1.778" layer="96" rot="R270"/>
+<attribute name="PN" x="101.6" y="58.42" size="1.778" layer="96" rot="R180" display="off"/>
 </instance>
 <instance part="L1" gate="G$1" x="73.66" y="83.82" rot="R90">

Commit message: fixed cap packages (5mm)
Parts:
- C10, C2, C3, C6, C7, C8, C9: device SparkFun-Passives:CAPPTH -> SparkFun-Passives:CAPPTH1
Changed lines of the file:
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@@
 <grid distance="0.1" unitdist="inch" unit="inch" style="lines" multiple="1" display="no" altdistance="0.01" altunitdist="inch" altunit="inch"/>
 <layers>
-<layer number="1" name="Top" color="4" fill="1" visible="no" active="no"/>
-<layer number="16" name="Bottom" color="1" fill="1" visible="no" active="no"/>
-<layer number="17" name="Pads" color="2" fill="1" visible="no" active="no"/>
-<layer number="18" name="Vias" color="2" fill="1" visible="no" active="no"/>
-<layer number="19" name="Unrouted" color="6" fill="1" visible="no" active="no"/>
-<layer number="20" name="Dimension" color="15" fill="1" visible="no" active="no"/>
-<layer number="21" name="tPlace" color="7" fill="1" visible="no" active="no"/>
-<layer number="22" name="bPlace" color="7" fill="1" visible="no" active="no"/>
-<layer number="23" name="tOrigins" color="15" fill="1" visible="no" active="no"/>
-<layer number="24" name="bOrigins" color="15" fill="1" visible="no" active="no"/>
-<layer number="25" name="tNames" color="7" fill="1" visible="no" active="no"/>
-<layer number="26" name="bNames" color="7" fill="1" visible="no" active="no"/>
-<layer number="27" name="tValues" color="7" fill="1" visible="no" active="no"/>
-<layer number="28" name="bValues" color="7" fill="1" visible="no" active="no"/>
+<layer number="1" name="Top" color="4" fill="1" visible="yes" active="no"/>
+<layer number="16" name="Bottom" color="1" fill="1" visible="yes" active="no"/>
+<layer number="17" name="Pads" color="2" fill="1" visible="yes" active="no"/>
+<layer number="18" name="Vias" color="2" fill="1" visible="yes" active="no"/>
+<layer number="19" name="Unrouted" color="6" fill="1" visible="yes" active="no"/>
+<layer number="20" name="Dimension" color="15" fill="1" visible="yes" active="no"/>
+<layer number="21" name="tPlace" color="14" fill="1" visible="yes" active="no"/>
+<layer number="22" name="bPlace" color="14" fill="1" visible="yes" active="no"/>
+<layer number="23" name="tOrigins" color="15" fill="1" visible="yes" active="no"/>
+<layer number="24" name="bOrigins" color="15" fill="1" visible="yes" active="no"/>
+<layer number="25" name="tNames" color="14" fill="1" visible="yes" active="no"/>
+<layer number="26" name="bNames" color="14" fill="1" visible="yes" active="no"/>
+<layer number="27" name="tValues" color="14" fill="1" visible="yes" active="no"/>
+<layer number="28" name="bValues" color="14" fill="1" visible="yes" active="no"/>
 <layer number="29" name="tStop" color="7" fill="3" visible="no" active="no"/>
 <layer number="30" name="bStop" color="7" fill="6" visible="no" active="no"/>
@@
 <layer number="35" name="tGlue" color="7" fill="4" visible="no" active="no"/>
 <layer number="36" name="bGlue" color="7" fill="5" visible="no" active="no"/>
-<layer number="37" name="tTest" color="7" fill="1" visible="no" active="no"/>
-<layer number="38" name="bTest" color="7" fill="1" visible="no" active="no"/>
+<layer number="37" name="tTest" color="7" fill="1" visible="yes" active="no"/>
+<layer number="38" name="bTest" color="7" fill="1" visible="yes" active="no"/>
 <layer number="39" name="tKeepout" color="4" fill="11" visible="no" active="no"/>
 <layer number="40" name="bKeepout" color="1" fill="11" visible="no" active="no"/>
@@
 <layer number="44" name="Drills" color="7" fill="1" visible="no" active="no"/>
 <layer number="45" name="Holes" color="7" fill="1" visible="no" active="no"/>
-<layer number="46" name="Milling" color="3" fill="1" visible="no" active="no"/>
-<layer number="47" name="Measures" color="7" fill="1" visible="no" active="no"/>
-<layer number="48" name="Document" color="7" fill="1" visible="no" active="no"/>
-<layer number="49" name="Reference" color="7" fill="1" visible="no" active="no"/>
-<layer number="50" name="dxf" color="7" fill="1" visible="no" active="no"/>
-<layer number="51" name="tDocu" color="7" fill="1" visible="no" active="no"/>
-<layer number="52" name="bDocu" color="7" fill="1" visible="no" active="no"/>
-<layer number="53" name="tGND_GNDA" color="7" fill="9" visible="no" active="no"/>
-<layer number="54" name="bGND_GNDA" color="1" fill="9" visible="no" active="no"/>
-<layer number="56" name="wert" color="7" fill="1" visible="no" active="no"/>
-<layer number="57" name="tCAD" color="7" fill="1" visible="no" active="no"/>
-<layer number="59" name="tCarbon" color="7" fill="1" visible="no" active="no"/>
-<layer number="60" name="bCarbon" color="7" fill="1" visible="no" active="no"/>
+<layer number="46" name="Milling" color="3" fill="1" visible="yes" active="no"/>
+<layer number="47" name="Measures" color="7" fill="1" visible="yes" active="no"/>
+<layer number="48" name="Document" color="7" fill="1" visible="yes" active="no"/>
+<layer number="49" name="Reference" color="7" fill="1" visible="yes" active="no"/>
+<layer number="50" name="dxf" color="7" fill="1" visible="yes" active="no"/>
+<layer number="51" name="tDocu" color="14" fill="1" visible="yes" active="no"/>
+<layer number="52" name="bDocu" color="14" fill="1" visible="yes" active="no"/>
+<layer number="53" name="tGND_GNDA" color="7" fill="9" visible="yes" active="no"/>
+<layer number="54" name="bGND_GNDA" color="1" fill="9" visible="yes" active="no"/>
+<layer number="56" name="wert" color="7" fill="1" visible="yes" active="no"/>
+<layer number="57" name="tCAD" color="7" fill="1" visible="yes" active="no"/>
+<layer number="59" name="tCarbon" color="7" fill="1" visible="yes" active="no"/>
+<layer number="60" name="bCarbon" color="7" fill="1" visible="yes" active="no"/>
 <layer number="90" name="Modules" color="5" fill="1" visible="yes" active="yes"/>
 <layer number="91" name="Nets" color="2" fill="1" visible="yes" active="yes"/>
@@
 <part name="SUPPLY13" library="SparkFun-Aesthetics" deviceset="5V" device=""/>
 <part name="GND12" library="SparkFun-Aesthetics" deviceset="GND" device=""/>
-<part name="C7" library="SparkFun-Passives" deviceset="CAP" device="PTH" value="10uF">
+<part name="C7" library="SparkFun-Passives" deviceset="CAP" device="PTH1" value="10uF">
 <attribute name="PN" value="445-173437-1-ND"/>
 </part>
-<part name="C8" library="SparkFun-Passives" deviceset="CAP" device="PTH" value="10uF">
+<part name="C8" library="SparkFun-Passives" deviceset="CAP" device="PTH1" value="10uF">
 <attribute name="PN" value="445-173437-1-ND"/>
 </part>
@@
 <attribute name="PN" value="1572-1306-ND"/>
 </part>
-<part name="C2" library="SparkFun-Passives" deviceset="CAP" device="PTH" value="0.1uf">
+<part name="C2" library="SparkFun-Passives" deviceset="CAP" device="PTH1" value="0.1uf">
 <attribute name="PN" value="BC2665CT-ND"/>
 </part>
-<part name="C3" library="SparkFun-Passives" deviceset="CAP" device="PTH" value="0.1uf">
+<part name="C3" library="SparkFun-Passives" deviceset="CAP" device="PTH1" value="0.1uf">
 <attribute name="PN" value="BC2665CT-ND"/>
 </part>
@@
 <attribute name="PN" value="1.00MXBK-ND"/>
 </part>
-<part name="C6" library="SparkFun-Passives" deviceset="CAP" device="PTH" value="0.1uf">
+<part name="C6" library="SparkFun-Passives" deviceset="CAP" device="PTH1" value="0.1uf">
 <attribute name="PN" value="445-173449-1-ND"/>
 </part>
@@
 <attribute name="PN" value="31.6KXBK-ND"/>
 </part>
-<part name="C10" library="SparkFun-Passives" deviceset="CAP" device="PTH" value="0.1uf">
+<part name="C10" library="SparkFun-Passives" deviceset="CAP" device="PTH1" value="0.1uf">
 <attribute name="PN" value="BC2665CT-ND"/>
 </part>
-<part name="C9" library="SparkFun-Passives" deviceset="CAP" device="PTH" value="0.1uf">
+<part name="C9" library="SparkFun-Passives" deviceset="CAP" device="PTH1" value="0.1uf">
 <attribute name="PN" value="BC2665CT-ND"/>
 </part>
